Commit message: robot model with friction ok, effective mass on EE ok

File: franka_description/robots/common/panda_arm.xacro (robot description, xacro)
@@ -35,4 +35,9 @@
         </geometry>
       </collision>
+      <inertial>
+        <mass value="0.629769" />
+        <origin xyz="-0.041018 -0.00014 0.049974" rpy="0 0 0" />
+        <inertia ixx="0.00315" ixy="8.2904e-07" ixz="0.00015" iyy="0.00388" iyz="8.2299e-06" izz="0.004285" />
+      </inertial>
     </link>
     <link name="${arm_id}_link1">
@@ -60,4 +65,9 @@
         </geometry>
       </collision>
+      <inertial>
+        <mass value="4.970684" />
+        <origin xyz="0.003875 0.002081 0.0" rpy="0 0 0" />
+        <inertia ixx="0.70337" ixy="-0.000139" ixz="0.006772" iyy="0.70661" iyz="0.019169" izz="0.009117" />
+      </inertial>
     </link>
     <joint name="${arm_id}_joint1" type="revolute">
@@ -93,4 +103,9 @@
         </geometry>
       </collision>
+      <inertial>
+        <mass value="0.646926" />
+        <origin xyz="-0.003141 -0.02872 0.003495" rpy="0 0 0" />
+        <inertia ixx="0.007962" ixy="-0.003925" ixz="0.010254" iyy="0.02811" iyz="0.000704" izz="0.025995" />
+      </inertial>
     </link>
     <joint name="${arm_id}_joint2" type="revolute">
@@ -126,4 +141,9 @@
         </geometry>
       </collision>
+      <inertial>
+        <mass value="3.228604" />
+        <origin xyz="0.027518 0.039252 -0.066502" rpy="0 0 0" />
+        <inertia ixx="0.037242" ixy="-0.004761" ixz="-0.011396" iyy="0.036155" iyz="-0.012805" izz="0.01083" />
+      </inertial>
     </link>
     <joint name="${arm_id}_joint3" type="revolute">
@@ -159,4 +179,9 @@
         </geometry>
       </collision>
+      <inertial>
+        <mass value="3.587895" />
+        <origin xyz="-0.05317 0.104419 0.027454" rpy="0 0 0" />
+        <inertia ixx="0.025853" ixy="0.007796" ixz="-0.001332" iyy="0.019552" iyz="0.008641" izz="0.028323" />
+      </inertial>
     </link>
     <joint name="${arm_id}_joint4" type="revolute">
@@ -210,4 +235,9 @@
         </geometry>
       </collision>
+      <inertial>
+        <mass value="1.225946" />
+        <origin xyz="-0.011953 0.041065 -0.038437" rpy="0 0 0" />
+        <inertia ixx="0.035549" ixy="-0.002117" ixz="-0.004037" iyy="0.029474" iyz="0.000229" izz="0.008627" />
+      </inertial>
     </link>
     <joint name="${arm_id}_joint5" type="revolute">
@@ -243,4 +273,9 @@
         </geometry>
       </collision>
+      <inertial>
+        <mass value="1.666555" />
+        <origin xyz="0.060149 -0.014117 -0.010517" rpy="0 0 0" />
+        <inertia ixx="0.001964" ixy="0.000109" ixz="-0.001158" iyy="0.004354" iyz="0.000341" izz="0.005433" />
+      </inertial>
     </link>
     <joint name="${arm_id}_joint6" type="revolute">
@@ -276,4 +311,9 @@
         </geometry>
       </collision>
+      <inertial>
+        <mass value="0.735522" />
+        <origin xyz="0.010517 -0.004252 0.061597" rpy="0 0 0" />
+        <inertia ixx="0.012516" ixy="-0.000428" ixz="-0.001196" iyy="0.010027" iyz="-0.000741" izz="0.004815" />
+      </inertial>
     </link>
     <joint name="${arm_id}_joint7" type="revolute">
